File: pcb/dw-probe-v1.1.sch (EAGLE design)
At the start: 23 parts, among them IC1 74LVC1G125DBV, IC2 74LVC1G125DBV, IC3 74LVC1G125DBV, IC4 TS1117BCW33_RPG, Q1 BSS138, Q2 IRLML6402, Q3 IRLML6402

Commit message: V1.1.11
Parts:
- removed MICRO, RX-IC: (no value), pinhead:PINHD-1X2
Connections:
- removed net N$21: RX-IC.2, U$1.3V
- removed net N$23: MICRO.2, U$1.D4*
- net N$22: no longer MICRO.1, RX-IC.1
Changed lines of the file:
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@@
 <part name="P+1" library="supply1" library_urn="urn:adsk.eagle:library:371" deviceset="VCC" device=""/>
 <part name="IC3" library="74xx-little-us" library_urn="urn:adsk.eagle:library:87" deviceset="74*1G125" device="DBV" package3d_urn="urn:adsk.eagle:package:2406/1" technology="LVC"/>
-<part name="RX-IC" library="pinhead" library_urn="urn:adsk.eagle:library:325" deviceset="PINHD-1X2" device="" package3d_urn="urn:adsk.eagle:package:22435/2"/>
 <part name="C3" library="rcl" library_urn="urn:adsk.eagle:library:334" deviceset="C-EU" device="C0805" package3d_urn="urn:adsk.eagle:package:23617/2" value="10uF"/>
 <part name="GND2" library="supply1" library_urn="urn:adsk.eagle:library:371" deviceset="GND" device=""/>
-<part name="MICRO" library="pinhead" library_urn="urn:adsk.eagle:library:325" deviceset="PINHD-1X2" device="" package3d_urn="urn:adsk.eagle:package:22435/2"/>
 </parts>
 <sheets>
@@
 <attribute name="VALUE" x="152.4" y="30.48" size="1.778" layer="96" rot="MR0"/>
 </instance>
-<instance part="RX-IC" gate="G$1" x="22.86" y="78.74" smashed="yes" rot="R180">
-<attribute name="NAME" x="29.21" y="73.025" size="1.778" layer="95" rot="R180"/>
-<attribute name="VALUE" x="29.21" y="83.82" size="1.778" layer="96" rot="R180"/>
-</instance>
 <instance part="C3" gate="G$1" x="88.9" y="27.94" smashed="yes" rot="R90">
 <attribute name="NAME" x="88.519" y="29.464" size="1.778" layer="95" rot="R90"/>
@@
 <instance part="GND2" gate="1" x="93.98" y="25.4" smashed="yes">
 <attribute name="VALUE" x="91.44" y="22.86" size="1.778" layer="96"/>
-</instance>
-<instance part="MICRO" gate="G$1" x="104.14" y="25.4" smashed="yes" rot="R270">
-<attribute name="NAME" x="102.87" y="20.955" size="1.778" layer="95"/>
-<attribute name="VALUE" x="99.06" y="31.75" size="1.778" layer="96" rot="R270"/>
 </instance>
 </instances>
@@
 </segment>
 </net>
-<net name="N$21" class="0">
-<segment>
-<pinref part="U$1" gate="G$1" pin="3V"/>
-<pinref part="RX-IC" gate="G$1" pin="2"/>
-<wire x1="45.72" y1="78.74" x2="25.4" y2="78.74" width="0.1524" layer="91"/>
-</segment>
-</net>
 <net name="N$22" class="0">
 <segment>
@@
 <junction x="40.64" y="66.04"/>
 <wire x1="40.64" y1="76.2" x2="40.64" y2="66.04" width="0.1524" layer="91"/>
-<pinref part="RX-IC" gate="G$1" pin="1"/>
-<wire x1="25.4" y1="76.2" x2="40.64" y2="76.2" width="0.1524" layer="91"/>
-<junction x="40.64" y="76.2"/>
 <pinref part="R2" gate="G$1" pin="1"/>
 <wire x1="86.36" y1="71.12" x2="101.6" y2="71.12" width="0.1524" layer="91"/>
@@
 <wire x1="101.6" y1="60.96" x2="101.6" y2="71.12" width="0.1524" layer="91"/>
 <junction x="101.6" y="71.12"/>
-<pinref part="MICRO" gate="G$1" pin="1"/>
-<wire x1="106.68" y1="27.94" x2="106.68" y2="60.96" width="0.1524" layer="91"/>
-<junction x="106.68" y="60.96"/>
-</segment>
-</net>
-<net name="N$23" class="0">
-<segment>
-<pinref part="U$1" gate="G$1" pin="D4*"/>
-<wire x1="81.28" y1="60.96" x2="99.06" y2="60.96" width="0.1524" layer="91"/>
-<wire x1="99.06" y1="60.96" x2="99.06" y2="27.94" width="0.1524" layer="91"/>
-<pinref part="MICRO" gate="G$1" pin="2"/>
-<wire x1="99.06" y1="27.94" x2="104.14" y2="27.94" width="0.1524" layer="91"/>
-</segment>
-</net>
+</segment>
+</net>
