File: pcb/dw-shield-V1.1.brd (EAGLE design)
At the start: 68.6 x 53.3 mm, 28 parts, among them IC1 74LVC1G125DBV, IC2 74LVC1G125DBV, IC3 74LVC1G125DBV, IC4 TS1117BCW33_RPG, Q1 BSS138, Q2 IRLML6402, Q3 IRLML6402

Commit message: V1.1.11
Parts:
- removed ICP-RX: (no value), pinhead:1X02
Connections:
- net N$2: no longer ICP-RX.2
- net N$20: no longer ICP-RX.1
Routing:
- net N$2: track 63.8 -> 43.7 mm
- net N$20: track 51.9 -> 46.1 mm
Changed lines of the file:
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@@
 <attribute name="SPICEPREFIX" value="C" x="33.02" y="12.065" size="1.778" layer="27" rot="R90" display="off"/>
-</element>
-<element name="ICP-RX" library="pinhead" library_urn="urn:adsk.eagle:library:325" package="1X02" package3d_urn="urn:adsk.eagle:package:22435/2" value="" x="58.42" y="41.275" smashed="yes">
-<attribute name="NAME" x="55.8038" y="43.1038" size="1.27" layer="25" ratio="10"/>
-<attribute name="POPULARITY" value="98" x="58.42" y="41.275" size="1.778" layer="27" display="off"/>
-<attribute name="VALUE" x="55.88" y="38.1" size="1.27" layer="27"/>
 </element>
 <element name="MEGA-INP" library="pinhead" library_urn="urn:adsk.eagle:library:325" package="1X01" package3d_urn="urn:adsk.eagle:package:22485/2" value="" x="59.69" y="32.385" smashed="yes">
@@
 <contactref element="R2" pad="1"/>
 <contactref element="MEGA-INP" pad="1"/>
-<contactref element="ICP-RX" pad="2"/>
 <wire x1="40.9575" y1="38.4175" x2="39.37" y2="36.83" width="0.2032" layer="1"/>
 <wire x1="40.9575" y1="50.165" x2="40.9575" y2="38.4175" width="0.2032" layer="1"/>
@@
 <wire x1="39.37" y1="36.83" x2="39.218" y2="36.83" width="0.2032" layer="1"/>
 <wire x1="41.5925" y1="50.8" x2="41.656" y2="50.8" width="0.2032" layer="1"/>
-<wire x1="59.69" y1="41.275" x2="59.69" y2="32.385" width="0.2032" layer="16"/>
 <wire x1="51.1175" y1="38.735" x2="49.8475" y2="37.465" width="0.2032" layer="1"/>
 <wire x1="51.1175" y1="48.5775" x2="51.1175" y2="38.735" width="0.2032" layer="1"/>
@@
 <wire x1="51.7525" y1="49.2125" x2="51.1175" y2="48.5775" width="0.2032" layer="1"/>
 <wire x1="49.8475" y1="37.465" x2="49.6" y2="37.465" width="0.2032" layer="1"/>
-<wire x1="51.7525" y1="49.2125" x2="59.69" y2="41.275" width="0.2032" layer="1"/>
 <wire x1="44.1325" y1="48.5775" x2="41.91" y2="50.8" width="0.2032" layer="16"/>
 <wire x1="51.1175" y1="48.5775" x2="44.1325" y2="48.5775" width="0.2032" layer="16"/>
 <wire x1="53.34" y1="50.8" x2="51.1175" y2="48.5775" width="0.2032" layer="16"/>
 <wire x1="41.91" y1="50.8" x2="41.656" y2="50.8" width="0.2032" layer="16"/>
+<wire x1="49.6" y1="37.465" x2="59.69" y2="32.385" width="0" layer="19" extent="1-1"/>
 </signal>
 <signal name="VCC">
@@
 </signal>
 <signal name="N$20">
-<contactref element="ICP-RX" pad="1"/>
 <contactref element="IOL" pad="2"/>
 <contactref element="JP4" pad="4"/>
@@
 <wire x1="46.99" y1="37.465" x2="31.115" y2="37.465" width="0.2032" layer="16"/>
 <wire x1="50.8" y1="41.275" x2="46.99" y2="37.465" width="0.2032" layer="16"/>
-<wire x1="57.15" y1="41.275" x2="51.435" y2="41.275" width="0.2032" layer="16"/>
 <wire x1="51.435" y1="41.275" x2="50.8" y2="41.275" width="0.2032" layer="16"/>
 <wire x1="51.435" y1="41.275" x2="60.96" y2="50.8" width="0.2032" layer="16"/>
