File: pcb/dw-shield-V1.1.sch (EAGLE design)
At the start: 28 parts, among them IC1 74LVC1G125DBV, IC2 74LVC1G125DBV, IC3 74LVC1G125DBV, IC4 TS1117BCW33_RPG, Q1 BSS138, Q2 IRLML6402, Q3 IRLML6402

Commit message: V1.1.11
Parts:
- removed ICP-RX: (no value), pinhead:PINHD-1X2
Connections:
- net N$2: no longer ICP-RX.2
- net N$20: no longer ICP-RX.1
Changed lines of the file:
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@@
 <part name="GND7" library="supply1" library_urn="urn:adsk.eagle:library:371" deviceset="GND" device=""/>
 <part name="C3" library="rcl" library_urn="urn:adsk.eagle:library:334" deviceset="C-EU" device="C1206" package3d_urn="urn:adsk.eagle:package:23618/2" value="10µF"/>
-<part name="ICP-RX" library="pinhead" library_urn="urn:adsk.eagle:library:325" deviceset="PINHD-1X2" device="" package3d_urn="urn:adsk.eagle:package:22435/2"/>
 <part name="MEGA-INP" library="pinhead" library_urn="urn:adsk.eagle:library:325" deviceset="PINHD-1X1" device="" package3d_urn="urn:adsk.eagle:package:22485/2"/>
 <part name="P+2" library="supply1" library_urn="urn:adsk.eagle:library:371" deviceset="VCC" device=""/>
@@
 <text x="215.265" y="36.83" size="1.778" layer="91" grouprefs="IOL1 IO PINS">6</text>
 <text x="215.265" y="39.37" size="1.778" layer="91" grouprefs="IOL1 IO PINS">7</text>
-<text x="215.265" y="50.8" size="1.778" layer="91" grouprefs="LABH PINS IO">8</text>
-<text x="215.265" y="53.34" size="1.778" layer="91" grouprefs="LABH PINS IO">9</text>
-<text x="215.265" y="55.88" size="1.778" layer="91" grouprefs="LABH PINS IO">10</text>
+<text x="215.265" y="50.8" size="1.778" layer="91" grouprefs="PINS LABH IO">8</text>
+<text x="215.265" y="53.34" size="1.778" layer="91" grouprefs="PINS LABH IO">9</text>
+<text x="215.265" y="55.88" size="1.778" layer="91" grouprefs="PINS LABH IO">10</text>
 <text x="215.265" y="58.42" size="1.778" layer="91" grouprefs="PINS IO">11</text>
-<text x="215.265" y="60.96" size="1.778" layer="91" grouprefs="LABH PINS IO">12</text>
-<text x="215.265" y="63.5" size="1.778" layer="91" grouprefs="LABH PINS IO">13</text>
+<text x="215.265" y="60.96" size="1.778" layer="91" grouprefs="PINS LABH IO">12</text>
+<text x="215.265" y="63.5" size="1.778" layer="91" grouprefs="PINS LABH IO">13</text>
 <text x="215.265" y="66.04" size="1.778" layer="91" grouprefs="PINS IO">GND</text>
 <text x="215.265" y="68.58" size="1.778" layer="91" grouprefs="PINS IO">REF</text>
@@
 <attribute name="VALUE" x="199.644" y="93.091" size="1.778" layer="96"/>
 </instance>
-<instance part="ICP-RX" gate="G$1" x="172.72" y="27.94" smashed="yes" rot="R180">
-<attribute name="NAME" x="179.07" y="22.225" size="1.778" layer="95" rot="R180"/>
-<attribute name="VALUE" x="179.07" y="33.02" size="1.778" layer="96" rot="R180"/>
-</instance>
 <instance part="MEGA-INP" gate="G$1" x="128.27" y="49.53" smashed="yes" rot="R90">
 <attribute name="NAME" x="125.095" y="43.18" size="1.778" layer="95" rot="R90"/>
@@
 <wire x1="128.27" y1="46.99" x2="128.27" y2="40.64" width="0.1524" layer="91"/>
 <junction x="128.27" y="40.64"/>
-<pinref part="ICP-RX" gate="G$1" pin="2"/>
-<wire x1="175.26" y1="27.94" x2="176.53" y2="27.94" width="0.1524" layer="91"/>
-<wire x1="176.53" y1="27.94" x2="176.53" y2="40.64" width="0.1524" layer="91"/>
-<junction x="176.53" y="40.64"/>
 </segment>
 </net>
@@
 <net name="N$20" class="0">
 <segment>
-<pinref part="ICP-RX" gate="G$1" pin="1"/>
 <wire x1="209.55" y1="25.4" x2="176.53" y2="25.4" width="0.1524" layer="91"/>
 <pinref part="IOL" gate="A" pin="2"/>
