File: pcb/dw-link-probe-V2.brd (EAGLE design)
At the start: 68.6 x 53.3 mm, 27 parts, among them IC1 74LVC1G125DBV, IC2 74LVC1G125DBV, IC3 74LVC1G125DBV, IC4 TS1117BCW33_RPG, Q1 BSS138, Q2 IRLML6402, Q3 IRLML6402

Commit message: changelog ficed
Parts:
- removed IC2, IC3: 74LVC1G125DBV, 74xx-little-us:SOT23-5
- removed IC4: TS1117BCW33_RPG, TS1117BCW33_RPG:SOT230P700X190-4N
- removed JP4: (no value), pinhead:1X09
- removed MEGA-INP: (no value), pinhead:1X01
- removed SW1: (no value), special:EDG-03
- added DEBUG, RES_EN: CON_HEADER_1X02-PTH, dp_devices:M1X2
- added PULLUP: CON_HEADER_1X03-PTH, dp_devices:M1X3
- added R10, R11: 10M, rcl:R1206
- added R9: 10k, rcl:R1206
- added SUPPLY: CON_HEADER_1X04, dp_devices:M1X4
- IC1: value 74LVC1G125DBV -> TS1117BCW33_RPG; device 74xx-little-us:SOT23-5 -> TS1117BCW33_RPG:SOT230P700X190-4N
- R5: value 220 -> 4.7k
- R7: value 10k -> 4.7k
- R8: value 4.7k -> 220
- moved R5 44.5 mm to (50.0, 26.7)
- moved R7 44.2 mm to (49.9, 19.8)
- moved R1 32.7 mm to (9.40, 32.4), turned to 90 degrees
- moved R4 19.6 mm to (5.84, 17.3)
- moved IC1 17.8 mm to (37.6, 23.1), turned to 0 degrees
- moved Q2 12.3 mm to (26.2, 34.8)
- moved R8 5.53 mm to (18.2, 37.8), turned to 0 degrees
- moved Q3 2.42 mm to (13.8, 21.1)
- moved LED1 0.40 mm to (9.78, 42.4), turned to 180 degrees
- turned C3 to 270 degrees
Connections:
- removed net N$20: IOL.2, JP4.4
- removed net N$21: IOH.6, LED1.A
- removed net N$23: IOL.1, JP4.3
- removed net N$24: IOL.4, JP4.5
- removed net N$5 (its old number): IC2.4, ISP.4, JP4.7
- removed net N$7: IC2.2, IOH.3
- removed net VCC: IC1.5, IC2.5, IC3.5, ISP.2, JP4.9, Q1.1, Q2.3, Q3.3, R3.2
- new net N$17: IOL.5, R8.1, R9.1
- net GND: now also C3.1, DEBUG.1, IC1.1, IOL.6, POWER.4, R1.1, R10.1, R11.1, RES_EN.1, RES_EN.2; no longer AD.1, C3.2, IC1.3, IC2.3, IC3.2, IC3.3, IC4.1, JP4.1, R8.1, SW1.1, SW1.2
- net N$1: now also IC1.3, SUPPLY.4; no longer IC4.3, Q2.2, R1.2, R4.2
- net N$10: now also PULLUP.3, R3.2; no longer Q2.1, R5.2
- net N$11: now also IOH.5, ISP.1; no longer ISP.5, JP4.2, Q1.2, SW1.3
- net N$12: now also AD.3, IOH.6, ISP.3, R5.1; no longer R3.1, SW1.4
- net N$13: now also AD.4, IOH.4, ISP.4, R7.1; no longer IOL.6, SW1.6
- net N$14: now also Q3.2, R4.2, SUPPLY.2, SUPPLY.3; no longer IOL.3, SW1.5
- net N$15: now also IC1.2, IC1.4, SUPPLY.1; no longer IC4.2, IC4.4, Q3.2, R7.2
- net N$16: now also Q2.3, R10.2, R5.2, R7.2; no longer IOH.2, R4.1, R5.1
- net N$18: now also DEBUG.2, IOL.4; no longer IOL.8, R6.1, R7.1
- net N$19: now also C3.2; no longer C3.1
- net N$2: no longer IOL.5, MEGA-INP.1
- net N$22: now also R1.2; no longer R8.2
- net N$3: now also AD.6, ISP.5, Q1.2, R11.2, R3.1; no longer IC1.4, ISP.3, JP4.6
- net N$4: now also IOL.3, R4.1, R6.1; no longer IC3.1, ISP.1, JP4.8
- net N$6: now also AD.5, ISP.2, PULLUP.2, Q1.1, Q2.2, Q3.3, R9.2; no longer IC1.1, IC2.1, IOL.7
- net N$8: now also Q2.1, R8.2; no longer IC1.2, IOH.5
- net N$9: now also IOL.8, LED1.A; no longer IC3.4, IOH.4, R1.1
Routing:
- net VCC: track 127.0 -> 0.00 mm, vias 2 -> 0
- net N$23: track 71.8 -> 0.00 mm, vias 1 -> 0
- net N$17: track 0.00 -> 66.7 mm, vias 0 -> 1
- net N$6: track 44.2 -> 107.3 mm, vias 2 -> 0
- net N$8: track 57.3 -> 6.66 mm, vias 4 -> 2
- net N$5 (its old number): track 50.1 -> 0.00 mm, vias 2 -> 0
- net N$1: track 115.6 -> 66.7 mm, vias 5 -> 3
- net N$11: track 88.7 -> 41.7 mm, vias 3 -> 1
- net N$20: track 46.1 -> 0.00 mm
- net N$14: track 76.0 -> 31.3 mm, vias 3 -> 0
- net N$24: track 40.0 -> 0.00 mm
- net GND: track 146.3 -> 184.0 mm, vias 1 -> 2
- net N$3: track 63.1 -> 95.5 mm, vias 3 -> 2
- net N$7: track 31.8 -> 0.00 mm, vias 4 -> 0
- net N$18: track 71.6 -> 44.6 mm, vias 2 -> 1
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Other:
- board text added: "+"
- board text added: "-"
- board text added: "3.3V"
- board text added: "dw-link"
- board text added: "ext."
- board text added: "no"
- board text added: "probe V2.0"
- board text removed: "DEBTX"
- board text removed: "MISO"
- board text removed: "MOSI"
- board text removed: "RX"
- board text removed: "SCK"
- board text removed: "Shield V1.1"
- board text removed: "TX"
- board text removed: "Vcc"
- board text removed: "Von"
- board text removed: "dW"
- board text removed: "dw-probe"

Commit message: pcb fix
Parts:
- moved PULLUP 0.38 mm to (16.9, 15.5)
- renumbered RES_EN to RESDIS
Changed lines of the file:
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@@
 <text x="12.573" y="8.763" size="1.778" layer="25" rot="R180">3.3V</text>
 <text x="21.59" y="6.35" size="1.778" layer="25" rot="R180">ext.</text>
-<text x="15.748" y="16.764" size="1.778" layer="25" rot="R180">no</text>
+<text x="15.367" y="16.764" size="1.778" layer="25" rot="R180">no</text>
 <text x="12.573" y="41.402" size="1.778" layer="25" rot="R180">-</text>
 <text x="12.446" y="45.339" size="1.778" layer="25" rot="R180">+</text>
@@
 <attribute name="SPICEPREFIX" value="R" x="9.398" y="32.385" size="1.778" layer="27" rot="R90" display="off"/>
 </element>
-<element name="PULLUP" library="dp_devices" package="M1X3" value="CON_HEADER_1X03-PTH" x="17.272" y="15.494" smashed="yes">
-<attribute name="NAME" x="16.002" y="17.0815" size="1.27" layer="25" ratio="10"/>
+<element name="PULLUP" library="dp_devices" package="M1X3" value="CON_HEADER_1X03-PTH" x="16.891" y="15.494" smashed="yes">
+<attribute name="NAME" x="15.621" y="17.0815" size="1.27" layer="25" ratio="10"/>
 </element>
 <element name="SUPPLY" library="dp_devices" package="M1X4" value="CON_HEADER_1X04" x="14.351" y="7.874" smashed="yes">
@@
 <attribute name="NAME" x="58.166" y="12.6365" size="1.27" layer="25" ratio="10"/>
 </element>
-<element name="RES_EN" library="dp_devices" package="M1X2" value="CON_HEADER_1X02-PTH" x="50.292" y="11.049" smashed="yes">
-<attribute name="NAME" x="47.752" y="12.6365" size="1.27" layer="25" ratio="10"/>
+<element name="RESDIS" library="dp_devices" package="M1X2" value="CON_HEADER_1X02-PTH" x="50.292" y="11.049" smashed="yes">
+<attribute name="NAME" x="47.371" y="12.6365" size="1.27" layer="25" ratio="10"/>
 </element>
 <element name="R10" library="rcl" library_urn="urn:adsk.eagle:library:334" package="R1206" package3d_urn="urn:adsk.eagle:package:23540/2" value="10M" x="29.337" y="42.037" smashed="yes" rot="R90">
@@
 <contactref element="POWER" pad="5"/>
 <contactref element="POWER" pad="4"/>
-<contactref element="RES_EN" pad="2"/>
+<contactref element="RESDIS" pad="2"/>
 <contactref element="R10" pad="1"/>
 <contactref element="R11" pad="1"/>
@@
 <wire x1="38.227" y1="13.338" x2="38.227" y2="13.335" width="0.4064" layer="1"/>
 <contactref element="C3" pad="1"/>
-<contactref element="RES_EN" pad="1"/>
+<contactref element="RESDIS" pad="1"/>
 <wire x1="35.433" y1="12.319" x2="33.02" y2="12.319" width="0.2032" layer="1"/>
 <wire x1="36.83" y1="11.43" x2="35.941" y2="12.319" width="0.2032" layer="16"/>
@@
 <wire x1="15.24" y1="20.955" x2="14.893" y2="21.082" width="0.2032" layer="1"/>
 <wire x1="15.24" y1="20.955" x2="15.494" y2="20.955" width="0.2032" layer="1"/>
-<wire x1="19.685" y1="15.875" x2="19.685" y2="20.955" width="0.2032" layer="1"/>
-<wire x1="19.685" y1="15.875" x2="19.812" y2="15.494" width="0.2032" layer="1"/>
+<wire x1="19.685" y1="16.256" x2="19.685" y2="20.955" width="0.2032" layer="1"/>
+<wire x1="19.685" y1="16.256" x2="19.431" y2="15.494" width="0.2032" layer="1"/>
 <wire x1="60.96" y1="20.955" x2="60.96" y2="2.54" width="0.2032" layer="16"/>
 <wire x1="61.595" y1="21.59" x2="60.96" y2="20.955" width="0.2032" layer="16"/>
@@
 <wire x1="26.035" y1="25.4" x2="29.21" y2="28.575" width="0.2032" layer="1"/>
 <wire x1="26.035" y1="19.05" x2="26.035" y2="25.4" width="0.2032" layer="1"/>
-<wire x1="22.86" y1="15.875" x2="26.035" y2="19.05" width="0.2032" layer="1"/>
+<wire x1="24.003" y1="17.018" x2="26.035" y2="19.05" width="0.2032" layer="1"/>
 <wire x1="41.91" y1="31.75" x2="42.062" y2="31.75" width="0.2032" layer="1"/>
-<wire x1="22.86" y1="15.875" x2="22.352" y2="15.494" width="0.2032" layer="1"/>
+<wire x1="24.003" y1="17.018" x2="21.971" y2="15.494" width="0.2032" layer="1"/>
 </signal>
 <signal name="N$3">

Commit message: V2.2.0
Parts:
- added RESET: (no value), Ergaenzung:TASTER-9314_SMD
- moved Q3 2.44 mm to (12.7, 18.9)
- moved R9 2.13 mm to (20.1, 31.8)
- moved R1 1.78 mm to (9.40, 34.2)
Connections:
- net GND: now also RESET.3, RESET.4
- net N$19: now also RESET.1, RESET.2
Routing:
- net N$19: track 8.12 -> 43.2 mm, vias 1 -> 3
- net GND: track 184.0 -> 195.1 mm, vias 2 -> 3
- net N$17: track 66.7 -> 71.4 mm
- net N$22: track 7.10 -> 5.33 mm
- net N$14: track 31.3 -> 29.7 mm
Other:
- board text added: "probe V2.2"
- board text removed: "probe V2.0"
